Commit message: Recolored table and rename main directory

File: pilz_tutorial_1/urdf/my_first_application.xacro (robot description, xacro)
@@ -6,4 +6,8 @@
   <material name="yellow">
     <color rgba="1 1 0 1"/>
+  </material>
+  <!-- coloring from the table -->
+  <material name="grey">
+    <color rgba="0.75 0.75 0.75 1"/>
   </material>
   <!-- instantiate the robot -->
@@ -15,4 +19,5 @@
         <box size="0.6 1.2 0.05"/>
       </geometry>
+      <material name="grey"/>
     </visual>
   </link>

Commit message: fixup path of stl file

File: pilz_tutorial_1/urdf/my_first_application.xacro (robot description, xacro)
@@ -26,5 +26,5 @@
       <origin rpy="1.5708 0 0" xyz="0 -0.5 0"/>
       <geometry>
-        <mesh filename="package://pilz_tutorial_step_1/urdf/meshes/PNOZ.stl"
+        <mesh filename="package://pilz_tutorial_1/urdf/meshes/PNOZ.stl"
           scale="0.001 0.001 0.001"/>
       </geometry>
