Commit message: Path changed to pilz_tutorial and moved in sub directory

File: pilz_tutorial_1/pilz_tutorial/urdf/my_first_application.xacro (robot description, xacro)
@@ -26,5 +26,5 @@
       <origin rpy="1.5708 0 0" xyz="0 -0.5 0"/>
       <geometry>
-        <mesh filename="package://pilz_tutorial_1/urdf/meshes/PNOZ.stl"
+        <mesh filename="package://pilz_tutorial/urdf/meshes/PNOZ.stl"
           scale="0.001 0.001 0.001"/>
       </geometry>
