Commit message: Neues Tutorial erstellt (Tutorial 2)

File: pilz_tutorial_2/pilz_tutorial/urdf/my_first_application.xacro (robot description, xacro)
@@ -15,7 +15,7 @@
   <link name="table">
     <visual>
-      <origin rpy="0 0 0" xyz="0 -0.45 -0.03"/>
+      <origin rpy="0 0 0" xyz="0 0 -0.03"/>
       <geometry>
-        <box size="0.6 1.2 0.05"/>
+      <box size="0.6 1.2 0.05"/>
       </geometry>
       <material name="grey"/>
@@ -32,4 +32,6 @@
     </visual>
   </link>
+  <!-- Add the tcp (tutorial 2) -->
+  <link name="prbt_tcp"/>
   <joint name="table_joint" type="fixed">
     <parent link="table"/>
@@ -40,3 +42,9 @@
     <child link="pnoz"/>
   </joint>
+  <!-- connect the added tcp and the flange with a joint (tutorial 2)-->
+  <joint name="prbt_fixed_joint_tcp" type="fixed">
+    <origin rpy="0 0 0" xyz="0 0 0.05"/>
+    <parent link="prbt_flange"/>
+    <child link="prbt_tcp"/>
+  </joint>
 </robot>
