Commit message: example with two scanners in one urdf

File: psen_scan_v2_tutorials/urdf/two_scanners.urdf.xacro (robot description, xacro)
@@ -1,18 +1,25 @@
 <?xml version="1.0"?>
+<!-- %Tag(FULLTEXT)% -->
 <robot xmlns:xacro="http://ros.org/wiki/xacro" name="psen_scan">
-  <!-- Example on how to use the psen_scan scanner within your robots urdf -->
+  <!-- %Tag(IMPORT_WORLD)% -->
   <xacro:include filename="$(find psen_scan_v2)/urdf/psen_scan.urdf.xacro" />
-  <link name="fixed"/>
-  <joint name="scanner_1_mount_joint" type="fixed">
-    <parent link="fixed" />
+  <link name="world"/>
+  <!-- %EndTag(IMPORT_WORLD)% -->
+  <!-- %Tag(FIRST_SCANNER)% -->
+  <joint name="laser_1_world_joint" type="fixed">
+    <parent link="world" />
     <child link="laser_1_mount_link" />
-    <origin rpy="0 0 0" xyz="-1 0 0"/>
+    <origin rpy="0 0 ${-pi/2}" xyz="0 -1 0"/>
   </joint>
-  <joint name="scanner_2_mount_joint" type="fixed">
-    <parent link="fixed" />
+  <xacro:psen_scan prefix="laser_1" />
+  <!-- %EndTag(FIRST_SCANNER)% -->
+  <!-- %Tag(SECOND_SCANNER)% -->
+  <joint name="laser_2_world_joint" type="fixed">
+    <parent link="world" />
     <child link="laser_2_mount_link" />
-    <origin rpy="0 0 0" xyz="1 0 0"/>
+    <origin rpy="0 0 ${pi/2}" xyz="0 1 0"/>
   </joint>
-  <xacro:psen_scan prefix="laser_1" ros_topic="scan" />
-  <xacro:psen_scan prefix="laser_2" ros_topic="scan2" />
+  <xacro:psen_scan prefix="laser_2" />
+  <!-- %EndTag(SECOND_SCANNER)% -->
 </robot>
+<!-- %EndTag(FULLTEXT)% -->

Commit message: we call it map

File: psen_scan_v2_tutorials/urdf/two_scanners.urdf.xacro (robot description, xacro)
@@ -2,11 +2,11 @@
 <!-- %Tag(FULLTEXT)% -->
 <robot xmlns:xacro="http://ros.org/wiki/xacro" name="psen_scan">
-  <!-- %Tag(IMPORT_WORLD)% -->
+  <!-- %Tag(IMPORT_MAP)% -->
   <xacro:include filename="$(find psen_scan_v2)/urdf/psen_scan.urdf.xacro" />
-  <link name="world"/>
-  <!-- %EndTag(IMPORT_WORLD)% -->
+  <link name="map"/>
+  <!-- %EndTag(IMPORT_MAP)% -->
   <!-- %Tag(FIRST_SCANNER)% -->
-  <joint name="laser_1_world_joint" type="fixed">
-    <parent link="world" />
+  <joint name="laser_1_map_joint" type="fixed">
+    <parent link="map" />
     <child link="laser_1_mount_link" />
     <origin rpy="0 0 ${-pi/2}" xyz="0 -1 0"/>
@@ -15,6 +15,6 @@
   <!-- %EndTag(FIRST_SCANNER)% -->
   <!-- %Tag(SECOND_SCANNER)% -->
-  <joint name="laser_2_world_joint" type="fixed">
-    <parent link="world" />
+  <joint name="laser_2_map_joint" type="fixed">
+    <parent link="map" />
     <child link="laser_2_mount_link" />
     <origin rpy="0 0 ${pi/2}" xyz="0 1 0"/>

Commit message: changing map to base_link for actual robot feel

File: psen_scan_v2_tutorials/urdf/two_scanners.urdf.xacro (robot description, xacro)
@@ -4,9 +4,9 @@
   <!-- %Tag(IMPORT_MAP)% -->
   <xacro:include filename="$(find psen_scan_v2)/urdf/psen_scan.urdf.xacro" />
-  <link name="map"/>
+  <link name="base_link"/>
   <!-- %EndTag(IMPORT_MAP)% -->
   <!-- %Tag(FIRST_SCANNER)% -->
-  <joint name="laser_1_map_joint" type="fixed">
-    <parent link="map" />
+  <joint name="laser_1_base_link_joint" type="fixed">
+    <parent link="base_link" />
     <child link="laser_1_mount_link" />
     <origin rpy="0 0 ${-pi/2}" xyz="0 -1 0"/>
@@ -15,6 +15,6 @@
   <!-- %EndTag(FIRST_SCANNER)% -->
   <!-- %Tag(SECOND_SCANNER)% -->
-  <joint name="laser_2_map_joint" type="fixed">
-    <parent link="map" />
+  <joint name="laser_2_base_link_joint" type="fixed">
+    <parent link="base_link" />
     <child link="laser_2_mount_link" />
     <origin rpy="0 0 ${pi/2}" xyz="0 1 0"/>
